File: Hardware/flight_computer/FMU_Power.sch (KiCad schematic (older format))
At the start: 1 part

Commit message: added parts for DAN <3
Parts:
- U?: symbol openDrone_parts:MIC5332-SSYMT-TR -> flight_computer-rescue:MIC5332-SSYMT-TR-openDrone_parts
Changed lines of the file:
@@
 $EndDescr
 $Comp
-L openDrone_parts:MIC5332-SSYMT-TR U?
+L flight_computer-rescue:MIC5332-SSYMT-TR-openDrone_parts U?
 U 1 1 5F64A1F5
 P 1650 1750

Commit message: added more parts and datasheets
Parts:
- U?: symbol flight_computer-rescue:MIC5332-SSYMT-TR-openDrone_parts -> flight_computer-rescue:MIC5332-SSYMT-TR-openDrone_parts-flight_computer-rescue
Changed lines of the file:
@@
 $EndDescr
 $Comp
-L flight_computer-rescue:MIC5332-SSYMT-TR-openDrone_parts U?
+L flight_computer-rescue:MIC5332-SSYMT-TR-openDrone_parts-flight_computer-rescue U?
 U 1 1 5F64A1F5
 P 1650 1750
