File: Hardware/flight_computer/flight_computer.sch (KiCad schematic (older format))
At the start: 32 parts

Commit message: added components, rerranged things to slow down dan
Parts:
- removed C? (x2): C_0u1, Capacitors_SMD:C_0805, symbol openDrone_parts:C_0u1
- removed C?: C_10n, Capacitors_SMD:C_0805, symbol openDrone_parts:C_10n
- removed C? (x2): C_10u, Capacitors_SMD:C_0805, symbol openDrone_parts:C_10u
- removed C?: C_2u2, Capacitors_SMD:C_0805, symbol openDrone_parts:C_2u2
- removed C?: C_220u, drone_footprints:UWT0G221MCL6GS, symbol openDrone_parts:C_220u
- removed D?: D_Schottky_70V, Diodes_SMD:D_SOD-523, symbol openDrone_parts:D_Schottky_70V
- removed R?: R_100K, Resistors_SMD:R_0805, symbol openDrone_parts:R_100K
- removed R?: R_220, Resistors_SMD:R_0805, symbol openDrone_parts:R_220
- removed R?: R_1K, Resistors_SMD:R_0805, symbol openDrone_parts:R_1K
- removed U?: Buck_Converter_2, drone_footprints:TPS54335ADDA, symbol openDrone_parts:Buck_Converter_2
- removed U?: LP5907QMFX-3.3, TO_SOT_Packages_SMD:SOT-23-5, symbol openDrone_parts:LP5907QMFX-3.3
Connections:
- net labels removed: VBAT, VDD_5V_IN
- wire segments 176 -> 142
Other:
- note added: "BATTERY = VBAT\nBUCK CONVERTER OUTPUT (VDD_5V_BRICK) = VDD_5V_BUCK\nUSB POWER (VBUS) = VDD_5V_USB\nRADIO 5V (VDD_5V_RECEIVER) = VDD_5V_RADIO\nGENERAL 5V (VDD_5V_IN) = VDD_5V_IN\nTELEM/FRSKY (VDD_5V_PERIPH) = VDD_5V_TELEM\nSTM POWER (FMU_VDD_3V3) = VDD_3V3_STM\nSENSORS POWER (VDD_3V3_SENSORS) = VDD_3V3_SENSORS\nRADIO POWER (VDD_3V3_SPEKTRUM) = RADIO_VDD_3V3\n"
- note added: "SPI FRAM"
- note added: "STM RESET WATCHDOG"
- moved on the sheet: C?, J?, Q?, U?, Y?

Commit message: added more components, added buzzer, servo circuits, re-arranged some power
Parts:
- removed C? (x2): C_8p, Capacitors_SMD:C_0805, symbol openDrone_parts:C_8p
- removed Q?: PMOS_20V_0.4A, TO_SOT_Packages_SMD:SOT-323_SC-70, symbol openDrone_parts:PMOS_20V_0.4A
- removed Y?: Crystal_24MHZ, drone_footprints:NX3225SA-24.000M-STD-CSR-1, symbol openDrone_parts:Crystal_24MHZ
- added BZ1: Buzzer, drone_footprints:PT-2040PQ, symbol openDrone_parts:Buzzer
- added C1: C_0u1, Capacitors_SMD:C_0805, symbol openDrone_parts:C_0u1
- added C2, C4: C_8p, Capacitors_SMD:C_0805, symbol openDrone_parts:C_8p
- added C7: C_220u, drone_footprints:UWT0G221MCL6GS, symbol openDrone_parts:C_220u
- added D1, D2: D_Schottky_10V_3A, Diodes_SMD:D_SOD-323F, symbol openDrone_parts:D_Schottky_10V_3A
- added J1: Micro_USB, Connectors_USB:USB_Micro-B_Molex_47346-0001, symbol openDrone_parts:Micro_USB
- added J2: MicroSD_molex, drone_footprints:2908-05WB-MG, symbol openDrone_parts:MicroSD_molex
- added L1: L_55m, drone_footprints:RLB0913-563K, symbol openDrone_parts:L_55m
- added Q1, Q2: PMOS_20V_.76A, drone_footprints:NTA4151PT1G, symbol openDrone_parts:PMOS_20V_.76A
- added R1, R2: R_22, Resistors_SMD:R_0805, symbol openDrone_parts:R_22
- added R10: R_120, Resistors_SMD:R_0805, symbol openDrone_parts:R_120
- added R3: R_1K, Resistors_SMD:R_0805, symbol openDrone_parts:R_1K
- added R4: R_10K, Resistors_SMD:R_0805, symbol openDrone_parts:R_10K
- added R5, R6, R7, R8, R9: R_100K, Resistors_SMD:R_0805, symbol openDrone_parts:R_100K
- added Y1: Crystal_24MHZ, drone_footprints:NX3225SA-24.000M-STD-CSR-1, symbol openDrone_parts:Crystal_24MHZ
- gave numbers to parts that had none: 15
Connections:
- net labels added: VDD_3V3_STM, VDD_5V_IN, VDD_5V_TELEM, VDD_5V_USB
- net labels removed: FMU_VBAT
- wire segments 142 -> 185
- no-connect marks 0 -> 4
Other:
- note added: "BATTERY = VBAT\nBUCK CONVERTER OUTPUT (VDD_5V_BRICK) = VDD_5V_BUCK\nUSB POWER (VBUS) = VDD_5V_USB\nRADIO 5V (VDD_5V_RECEIVER) = VDD_5V_RADIO\nGENERAL 5V (VDD_5V_IN) = VDD_5V_IN\nTELEM/FRSKY (VDD_5V_PERIPH) = VDD_5V_AUX\nSTM POWER (FMU_VDD_3V3) = VDD_3V3_STM\nSENSORS POWER (VDD_3V3_SENSORS) = VDD_3V3_SENSORS\nRADIO POWER (VDD_3V3_SPEKTRUM) = VDD_3V3_RADIO\n"
- note added: "BUZZER"
- note removed: "BATTERY = VBAT\nBUCK CONVERTER OUTPUT (VDD_5V_BRICK) = VDD_5V_BUCK\nUSB POWER (VBUS) = VDD_5V_USB\nRADIO 5V (VDD_5V_RECEIVER) = VDD_5V_RADIO\nGENERAL 5V (VDD_5V_IN) = VDD_5V_IN\nTELEM/FRSKY (VDD_5V_PERIPH) = VDD_5V_TELEM\nSTM POWER (FMU_VDD_3V3) = VDD_3V3_STM\nSENSORS POWER (VDD_3V3_SENSORS) = VDD_3V3_SENSORS\nRADIO POWER (VDD_3V3_SPEKTRUM) = RADIO_VDD_3V3\n"
- moved on the sheet: C10, C11, C12, C13, C14, C15, C3, C5, C6, C8, C9, J3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

Commit message: Finishes v1 connections
Connections:
- net FMU_VDD_3V3: no longer C10.2, C11.2, C12.2, C14.2, C15.2, C6.2, C8.2, C9.2, U1.3 (~WP), U1.7 (~HOLD), U1.8 (Vdd), U2.100 (VDD), U2.11 (VDD), U2.19 (VDD), U2.21 (VREF+), U2.22 (VDDA), U2.28 (VDD), U2.50 (VDD), U2.75 (VDD)
- net VDD_3V3_STM: now also C10.2, C11.2, C12.2, C14.2, C15.2, C6.2, C8.2, C9.2, U1.3 (~WP), U1.7 (~HOLD), U1.8 (Vdd), U2.100 (VDD), U2.11 (VDD), U2.19 (VDD), U2.21 (VREF+), U2.22 (VDDA), U2.28 (VDD), U2.50 (VDD), U2.75 (VDD)
- net VDD_5V_SENSE: now reaches U2.24 (PA1)
- net VBAT_SENSE: now reaches U2.25 (PA2)
- net VDD_3V3_RADIO_EN: now reaches U2.34 (PC5)
- net BUZZER_CTRL: now reaches U2.35 (PB0)
- net BUZZER_CTRL: now also Q1.1 (G)
- net SPEKTRUM_POWER_CTRL: now reaches U2.4 (PE5)
- net RPI_POWER_CTRL: now reaches U2.5 (PE6)
- net RPI_POWER_CTRL: now also Q2.1 (G)
- net SERVO_CH1_GPIO: now reaches U2.81 (PD0)
- net SERVO_CH2_GPIO: now reaches U2.82 (PD1)
- net VDD_BUCK_VALID: now reaches U2.91 (PB5)
- net VBUS_VALID renamed VDD_USB_VALID
- net VDD_5V_TELEM renamed VDD_5V_AUX
Other:
- note added: "VBAT comes in from ESC"
Changed lines of the file:
@@
 Comment4 ""
 $EndDescr
-Text HLabel 8750 5700 2    50   Input ~ 0
-VBUS_VALID
 $Comp
 L openDrone_parts:FRAM_128K U1
@@
 	6800 10300 6800 10750
 Wire Wire Line
-	6700 6700 6950 6700
-Text HLabel 6800 9900 2    50   Input ~ 0
-FMU_VDD_3V3
-Wire Wire Line
 	7550 2000 7550 1950
 $Comp
@@
 $EndComp
 Connection ~ 7450 1800
-Text HLabel 8800 1800 2    50   Input ~ 0
-FMU_VDD_3V3
 Wire Wire Line
 	8800 1800 8650 1800
@@
 	1    0    0    -1
 $EndComp
-Wire Wire Line
-	6950 5100 6800 5100
-Wire Wire Line
-	6950 4900 6800 4900
-Wire Wire Line
-	6950 5300 6800 5300
-Wire Wire Line
-	6950 5400 6800 5400
-Text Label 6800 5400 2    50   ~ 0
+Text Label 6950 5400 2    50   ~ 0
 FMU_CH1
-Text Label 6800 5300 2    50   ~ 0
+Text Label 6950 5300 2    50   ~ 0
 FMU_CH2
-Text Label 6800 5100 2    50   ~ 0
+Text Label 6950 5100 2    50   ~ 0
 FMU_CH3
-Text Label 6800 4900 2    50   ~ 0
+Text Label 6950 4900 2    50   ~ 0
 FMU_CH4
-Text Label 1850 1100 0    50   ~ 0
+Text Label 1700 1100 0    50   ~ 0
 FMU_CH1
-Text Label 1850 1000 0    50   ~ 0
+Text Label 1700 1000 0    50   ~ 0
 FMU_CH2
-Text Label 1850 900  0    50   ~ 0
+Text Label 1700 900  0    50   ~ 0
 FMU_CH3
-Text Label 1850 800  0    50   ~ 0
+Text Label 1700 800  0    50   ~ 0
 FMU_CH4
-Wire Wire Line
-	1700 800  1850 800
-Wire Wire Line
-	1850 900  1700 900
-Wire Wire Line
-	1700 1000 1850 1000
-Wire Wire Line
-	1850 1100 1700 1100
-Text Label 6750 4700 2    50   ~ 0
+Text Label 6950 4700 2    50   ~ 0
 FMU_UART7_RX
-Text Label 6750 4800 2    50   ~ 0
+Text Label 6950 4800 2    50   ~ 0
 FMU_UART7_TX
-Wire Wire Line
-	6950 4700 6750 4700
-Wire Wire Line
-	6750 4800 6950 4800
-Text Label 1850 2700 0    50   ~ 0
+Text Label 1700 2700 0    50   ~ 0
 FMU_UART7_RX
-Text Label 1850 2800 0    50   ~ 0
+Text Label 1700 2800 0    50   ~ 0
 FMU_UART7_TX
-Text Label 6750 6000 2    50   ~ 0
+Text Label 6950 6000 2    50   ~ 0
 FMU_USART2_CTS
-Text Label 6750 6100 2    50   ~ 0
+Text Label 6950 6100 2    50   ~ 0
 FMU_USART2_RTS
-Text Label 6750 6200 2    50   ~ 0
+Text Label 6950 6200 2    50   ~ 0
 FMU_USART2_TX
 $Comp
@@
 	1    0    0    -1
 $EndComp
-Text Label 6750 6300 2    50   ~ 0
+Text Label 6950 6300 2    50   ~ 0
 FMU_USART2_RX
-Wire Wire Line
-	6750 6300 6950 6300
-Wire Wire Line
-	6950 6200 6750 6200
-Wire Wire Line
-	6750 6100 6950 6100
-Wire Wire Line
-	6950 6000 6750 6000
-Text Label 1850 1550 0    50   ~ 0
+Text Label 1700 1550 0    50   ~ 0
 FMU_USART2_CTS
-Text Label 1850 1650 0    50   ~ 0
+Text Label 1700 1650 0    50   ~ 0
 FMU_USART2_RTS
-Text Label 1850 1750 0    50   ~ 0
+Text Label 1700 1750 0    50   ~ 0
 FMU_USART2_TX
-Text Label 1850 1850 0    50   ~ 0
+Text Label 1700 1850 0    50   ~ 0
 FMU_USART2_RX
-Wire Wire Line
-	1700 1550 1850 1550
-Wire Wire Line
-	1850 1650 1700 1650
-Wire Wire Line
-	1700 1750 1850 1750
-Wire Wire Line
-	1850 1850 1700 1850
 Text Label 6950 4000 2    50   ~ 0
 FMU_USART8_RX
 Text Label 6950 4100 2    50   ~ 0
 FMU_USART8_TX
-Text Label 1850 2550 0    50   ~ 0
+Text Label 1700 2550 0    50   ~ 0
 FMU_USART8_RX
-Text Label 1850 2450 0    50   ~ 0
+Text Label 1700 2450 0    50   ~ 0
 FMU_USART8_TX
-Wire Wire Line
-	1700 2700 1850 2700
-Wire Wire Line
-	1700 2800 1850 2800
-Wire Wire Line
-	1700 2550 1850 2550
-Wire Wire Line
-	1850 2450 1700 2450
 Text Label 8750 5800 0    50   ~ 0
 RSSI_IN
-Text Label 1850 2250 0    50   ~ 0
+Text Label 1700 2250 0    50   ~ 0
 RSSI_IN
-Wire Wire Line
-	1700 2250 1850 2250
 Text Label 8750 2800 0    50   ~ 0
 SENSOR_SCK
@@
 F16 "SWCLK" I R 1700 3000 50
 F17 "SWDIO" I R 1700 3100 50
-F18 "3V3" I R 1700 2900 50
 F19 "FMU_USART8_TX" I R 1700 2450 50
 F20 "FMU_USART8_RX" I R 1700 2550 50
 F21 "FrSky_INV" I R 1700 3350 50
-F22 "VDD_5V_PERIPH" I R 1700 3450 50
-F23 "VDD_5V_RECEIVER" I R 1700 3550 50
-F24 "FMU_RC_OUTPUT" I R 1700 3650 50
-F25 "FMU_RC_INPUT" I R 1700 3750 50
-F26 "SBUS_INV" I R 1700 3850 50
+F22 "FMU_RC_OUTPUT" I R 1700 3650 50
+F23 "FMU_RC_INPUT" I R 1700 3750 50
+F24 "SBUS_INV" I R 1700 3850 50
+F25 "VDD_5V_RADIO" I R 1700 3450 50
+F26 "VDD_5V_AUX" I R 1700 3250 50
+F27 "SERVO_CH_1" I R 1700 4000 50
+F28 "SERVO_CH_2" I R 1700 4100 50
+F29 "VDD_3V3_RADIO" I R 1700 2100 50
+F30 "VDD_3V3_STM" I R 1700 2000 50
 $EndSheet
 Text Label 8750 2600 0    50   ~ 0
@@
 Text Label 8750 5500 0    50   ~ 0
 FRAM_MOSI
-Text Label 6700 6700 2    50   ~ 0
+Text Label 6950 6700 2    50   ~ 0
 FRAM_CS
 Text Label 5600 10200 2    50   ~ 0
@@
 F2 "VDD_3V3_SENSORS_EN" I R 1700 6550 50
 F3 "VDD_5V_IN" I R 1700 5200 50
-F4 "VDD_3V3_PERIPH_EN" I R 1700 6450 50
-F5 "SPEKTRUM_POWER" I R 1700 6650 50
-F6 "VDD_3V3_RADIO" I R 1700 5550 50
-F7 "VDD_5V_RADIO" I R 1700 5400 50
-F8 "VDD_5V_TELEM" I R 1700 5300 50
-F9 "VDD_5V_BUCK" I R 1700 5000 50
-F10 "VBAT" I R 1700 4700 50
-F11 "VDD_BUCK_VALID" I R 1700 6150 50
-F12 "VDD_5V_USB" I R 1700 4900 50
-F13 "VDD_USB_VALID" I R 1700 6250 50
-F14 "VBAT_SENSE" I R 1700 5950 50
-F15 "VDD_5V_SENSE" I R 1700 6050 50
-F16 "VDD_3V3_SENSORS" I R 1700 5650 50
-F18 "VDD_3V3_STM" I R 1700 5750 50
+F4 "VDD_3V3_RADIO" I R 1700 5550 50
+F5 "VDD_5V_RADIO" I R 1700 5400 50
+F6 "VBAT" I R 1700 4700 50
+F7 "VDD_BUCK_VALID" I R 1700 6150 50
+F8 "VDD_5V_USB" I R 1700 4900 50
+F9 "VDD_USB_VALID" I R 1700 6250 50
+F10 "VBAT_SENSE" I R 1700 5950 50
+F11 "VDD_5V_SENSE" I R 1700 6050 50
+F12 "VDD_3V3_SENSORS" I R 1700 5650 50
+F13 "VDD_3V3_STM" I R 1700 5750 50
+F14 "VDD_5V_AUX" I R 1700 5100 50
+F15 "SPEKTRUM_POWER_CTRL" I R 1700 6650 50
+F16 "VDD_3V3_RADIO_EN" I R 1700 6450 50
 $EndSheet
 Connection ~ 8850 10300
@@
 Text Label 14150 1350 2    50   ~ 0
 IMU_ACCEL_CS
-Text Label 14150 3050 2    50   ~ 0
+Text Label 1700 6550 0    50   ~ 0
 VDD_3V3_SENSORS_EN
 $Sheet
@@
 F7 "IMU_INT1_ACCEL" I L 14150 1550 50
 F8 "INT3_GYRO" I L 14150 1650 50
-F9 "VDDIO" I L 14150 1950 50
 F10 "MAG_SDO_SA1" I L 14150 2050 50
 F11 "MAG_DRDY" I L 14150 2150 50
@@
 F17 "BARO_MOSI" I L 14150 2850 50
 F18 "BARO_SCK" I L 14150 2950 50
-F19 "VDD_3V3_SENSORS_EN" I L 14150 3050 50
-F20 "VDD_5V" I L 14150 3150 50
-F21 "GPS_UART_TX" I L 14150 3250 50
-F22 "GPS_UART_RX" I L 14150 3350 50
+F19 "GPS_UART_TX" I L 14150 3250 50
+F20 "GPS_UART_RX" I L 14150 3350 50
+F21 "VDD_3V3_SENSORS" I L 14150 3100 50
 $EndSheet
 Entry Wire Line
@@
 	-1   0    0    -1
 $EndComp
-Text HLabel 6950 2900 0    50   Input ~ 0
-FMU_VDD_3V3
 Wire Wire Line
 	7100 1450 7450 1450
@@
 	6450 1950 6700 1950
 Connection ~ 6700 1950
-Text HLabel 5750 1950 0    50   Input ~ 0
-VDD_3V3_STM
 Wire Wire Line
 	6650 2500 6950 2500
@@
 Wire Wire Line
 	12950 6200 12850 6200
-Text HLabel 12850 6200 0    50   Input ~ 0
-VDD_5V_IN
 $Comp
 L openDrone_parts:D_Schottky_10V_3A D2
@@
 Wire Wire Line
 	10950 9650 10900 9650
-Text HLabel 10900 9650 0    50   Input ~ 0
-VDD_5V_TELEM
 $Comp
 L power:GND #PWR013
@@
 	1    0    0    -1
 $EndComp
-Text HLabel 4400 9100 0    50   Input ~ 0
-VDD_5V_USB
 Wire Wire Line
 	4900 8850 4750 8850
@@
 NoConn ~ 9950 9100
 NoConn ~ 9950 9300
+Text Label 6950 2900 2    50   ~ 0
+VDD_3V3_STM
+Text Label 5750 1950 2    50   ~ 0
+VDD_3V3_STM
+Text Label 8800 1800 0    50   ~ 0
+VDD_3V3_STM
+Text Label 14150 3100 2    50   ~ 0
+VDD_3V3_SENSORS
+Text Label 1700 5650 0    50   ~ 0
+VDD_3V3_SENSORS
+Text Label 1700 4900 0    50   ~ 0
+VDD_5V_USB
+Text Label 1700 5750 0    50   ~ 0
+VDD_3V3_STM
+Text Label 12850 6200 2    50   ~ 0
+VDD_5V_IN
+Text Label 1700 5200 0    50   ~ 0
+VDD_5V_IN
+Text Label 1700 6650 0    50   ~ 0
+SPEKTRUM_POWER_CTRL
+Text Label 6950 4500 2    50   ~ 0
+SPEKTRUM_POWER_CTRL
+Text Label 1700 6250 0    50   ~ 0
+VDD_USB_VALID
+Text Label 8750 5700 0    50   ~ 0
+VDD_USB_VALID
+Text Label 1700 6150 0    50   ~ 0
+VDD_BUCK_VALID
+Text Label 8750 4500 0    50   ~ 0
+VDD_BUCK_VALID
+Text Label 8750 2500 0    50   ~ 0
+VBAT_SENSE
+Text Label 1700 5950 0    50   ~ 0
+VBAT_SENSE
+Text Label 8750 2400 0    50   ~ 0
+VDD_5V_SENSE
+Text Label 1700 6050 0    50   ~ 0
+VDD_5V_SENSE
+Text Label 12650 6500 2    50   ~ 0
+RPI_POWER_CTRL
+Text Label 6950 4600 2    50   ~ 0
+RPI_POWER_CTRL
+Text Label 6800 9900 0    50   ~ 0
+VDD_3V3_STM
+Text Label 10900 9650 2    50   ~ 0
+VDD_5V_AUX
+Text Label 1700 5100 0    50   ~ 0
+VDD_5V_AUX
+Text Label 1700 3250 0    50   ~ 0
+VDD_5V_AUX
+Text Label 1700 1400 0    50   ~ 0
+VBAT
+Text Label 1700 4700 0    50   ~ 0
+VBAT
+Text Notes 2100 1400 0    50   ~ 0
+VBAT comes in from ESC
+Text Label 10350 10550 1    50   ~ 0
+BUZZER_CTRL
+Text Label 8750 4000 0    50   ~ 0
+BUZZER_CTRL
+Text Label 1700 3450 0    50   ~ 0
+VDD_5V_RADIO
+Text Label 1700 5400 0    50   ~ 0
+VDD_5V_RADIO
+Text Label 1700 5550 0    50   ~ 0
+VDD_3V3_RADIO
+Text Label 1700 2100 0    50   ~ 0
+VDD_3V3_RADIO
+Text Label 1700 2000 0    50   ~ 0
+VDD_3V3_STM
+Text Label 1700 6450 0    50   ~ 0
+VDD_3V3_RADIO_EN
+Text Label 8750 6200 0    50   ~ 0
+VDD_3V3_RADIO_EN
+Text Label 1700 4000 0    50   ~ 0
+SERVO_CH1_GPIO
+Text Label 1700 4100 0    50   ~ 0
+SERVO_CH2_GPIO
+Text Label 6950 5700 2    50   ~ 0
+SERVO_CH1_GPIO
+Text Label 6950 5800 2    50   ~ 0
+SERVO_CH2_GPIO
 $EndSCHEMATC
