File: Hardware/rev2/flight_computer/flight_computer.sch (KiCad schematic (older format))
At the start: 43 parts, among them J1 Micro_USB, J2 MicroSD_molex, J3 rpi_zero_w, Q2 PMOS_20V_.76A, SW1 Switch_SMT, U1 FRAM_128K, U2 STM32F427VITx, U3 MCP131T-300E_TT, Y1 Crystal_24MHZ

Commit message: Removes frysky + spektrum connectors
Connections:
- net FMU_USART8_RX: no longer names the net of U2.97 (PE0)
- net FMU_USART8_TX: no longer names the net of U2.98 (PE1)
- net FrSky_INV: no longer names the net of U2.69 (PA10)
- net RC_INPUT_USART1_RX: no longer names the net of U2.93 (PB7)
- net RC_OUTPUT_USART1_TX: no longer names the net of U2.92 (PB6)
- net RSSI_IN: no longer names the net of U2.37 (PB2)
- net SBUS_INV: no longer names the net of U2.36 (PB1)
- net VDD_3V3_RADIO_EN: no longer names the net of U2.34 (PC5)
Changed lines of the file:
@@
 Text Label 1700 1850 0    50   ~ 0
 FMU_USART2_RX
-Text Label 6950 4000 2    50   ~ 0
-FMU_USART8_RX
-Text Label 6950 4100 2    50   ~ 0
-FMU_USART8_TX
-Text Label 1700 2550 0    50   ~ 0
-FMU_USART8_RX
-Text Label 1700 2450 0    50   ~ 0
-FMU_USART8_TX
-Text Label 8750 4200 0    50   ~ 0
-RSSI_IN
-Text Label 1700 2250 0    50   ~ 0
-RSSI_IN
 Text Label 8750 2800 0    50   ~ 0
 SENSOR_SCK
@@
 F11 "cts_telem_1" I R 1700 1550 50
 F12 "rts_telem_1" I R 1700 1650 50
-F13 "rssi_in" I R 1700 2250 50
 F14 "FMU_UART7_RX" I R 1700 2700 50
 F15 "FMU_UART7_TX" I R 1700 2800 50
 F16 "SWCLK" I R 1700 3000 50
 F17 "SWDIO" I R 1700 3100 50
-F18 "FMU_USART8_TX" I R 1700 2450 50
-F19 "FMU_USART8_RX" I R 1700 2550 50
-F20 "FrSky_INV" I R 1700 3350 50
-F21 "FMU_RC_OUTPUT" I R 1700 3650 50
-F22 "FMU_RC_INPUT" I R 1700 3750 50
-F23 "SBUS_INV" I R 1700 3850 50
 F24 "VDD_5V_RADIO" I R 1700 3450 50
 F25 "VDD_5V_AUX" I R 1700 3250 50
 F26 "SERVO_CH_1" I R 1700 4000 50
 F27 "SERVO_CH_2" I R 1700 4100 50
-F28 "VDD_3V3_RADIO" I R 1700 2100 50
 F29 "VDD_3V3_STM" I R 1700 2000 50
 $EndSheet
@@
 Text Label 6950 5200 2    50   ~ 0
 MAG_DRDY
-Text Label 1700 3850 0    50   ~ 0
-SBUS_INV
-Text Label 8750 3300 0    50   ~ 0
-FrSky_INV
-Text Label 1700 3350 0    50   ~ 0
-FrSky_INV
-Text Label 8750 4700 0    50   ~ 0
-RC_INPUT_USART1_RX
-Text Label 8750 4600 0    50   ~ 0
-RC_OUTPUT_USART1_TX
-Text Label 1700 3750 0    50   ~ 0
-RC_INPUT_USART1_RX
-Text Label 1700 3650 0    50   ~ 0
-RC_OUTPUT_USART1_TX
 Text Label 8750 4800 0    50   ~ 0
 RASPI_I2C1_SCL
@@
 F2 "VDD_3V3_SENSORS_EN" I R 1700 6550 50
 F3 "VDD_5V_IN" I R 1700 5200 50
-F4 "VDD_3V3_RADIO" I R 1700 5550 50
 F5 "VDD_5V_RADIO" I R 1700 5400 50
 F6 "VBAT" I R 1700 4700 50
@@
 F13 "VDD_3V3_STM" I R 1700 5750 50
 F14 "VDD_5V_AUX" I R 1700 5100 50
-F15 "VDD_3V3_RADIO_EN" I R 1700 6450 50
 $EndSheet
 Text Notes 8500 11050 0    79   ~ 0
@@
 Text Label 1700 5400 0    50   ~ 0
 VDD_5V_RADIO
-Text Label 1700 5550 0    50   ~ 0
-VDD_3V3_RADIO
-Text Label 1700 2100 0    50   ~ 0
-VDD_3V3_RADIO
 Text Label 1700 2000 0    50   ~ 0
 VDD_3V3_STM
-Text Label 1700 6450 0    50   ~ 0
-VDD_3V3_RADIO_EN
-Text Label 8750 6200 0    50   ~ 0
-VDD_3V3_RADIO_EN
 Text Label 1700 4000 0    50   ~ 0
 SERVO_CH1_GPIO
@@
 DEBUG_LED_2
 NoConn ~ 6950 4500
-Text Label 8750 4100 0    50   ~ 0
-SBUS_INV
 Text Label 6950 6500 2    50   ~ 0
 DEBUG_LED_1

Commit message: Fix gps uart and update CubeMX config
Connections:
- net GPS_USART6_RX renamed STM_RX_GPS_TX_USART6
- net GPS_USART6_TX renamed STM_TX_GPS_RX_USART6
Changed lines of the file:
@@
 FRAM_MOSI
 Text Label 8750 6300 0    50   ~ 0
-GPS_USART6_TX
+STM_TX_GPS_RX_USART6
 Text Label 8750 6400 0    50   ~ 0
-GPS_USART6_RX
+STM_RX_GPS_TX_USART6
 Text Label 6950 5900 2    50   ~ 0
 SDIO_CMD
@@
 Text Label 8750 6500 0    50   ~ 0
 SDIO_D0
-Text Label 14150 3250 2    50   ~ 0
-GPS_USART6_TX
-Text Label 14150 3350 2    50   ~ 0
-GPS_USART6_RX
 Text Label 8750 3400 0    50   ~ 0
 OTG_FS_D_N
@@
 	8600 10650 8450 10650
 Connection ~ 8600 10650
+Text Label 14150 3350 2    50   ~ 0
+STM_TX_GPS_RX_USART6
+Text Label 14150 3250 2    50   ~ 0
+STM_RX_GPS_TX_USART6
 $EndSCHEMATC

Commit message: Fixes telemetry uart and dshot
Connections:
- net FMU_CH1: now also U2.40 (PE9); no longer U2.45 (PE14)
- net FMU_CH2: now also U2.42 (PE11); no longer U2.44 (PE13)
- net FMU_CH3: now also U2.44 (PE13); no longer U2.42 (PE11)
- net FMU_CH4: now also U2.45 (PE14); no longer U2.40 (PE9)
- net FMU_USART2_CTS renamed STM_CTS_TELEM_RTS_USART2
- net FMU_USART2_RTS renamed STM_RTS_TELEM_CTS_USART2
- net FMU_USART2_RX renamed STM_RX_TELEM_TX_USART2
- net FMU_USART2_TX renamed STM_TX_TELEM_RX_USART2
- no-connect marks 55 -> 63
Changed lines of the file:
@@
 	1    0    0    -1
 $EndComp
+Text Label 6950 4900 2    50   ~ 0
+FMU_CH1
+Text Label 6950 5100 2    50   ~ 0
+FMU_CH2
+Text Label 6950 5300 2    50   ~ 0
+FMU_CH3
 Text Label 6950 5400 2    50   ~ 0
-FMU_CH1
-Text Label 6950 5300 2    50   ~ 0
-FMU_CH2
-Text Label 6950 5100 2    50   ~ 0
-FMU_CH3
-Text Label 6950 4900 2    50   ~ 0
 FMU_CH4
 Text Label 1700 1100 0    50   ~ 0
@@
 Text Label 1700 2800 0    50   ~ 0
 FMU_UART7_TX
-Text Label 6950 6000 2    50   ~ 0
-FMU_USART2_CTS
-Text Label 6950 6100 2    50   ~ 0
-FMU_USART2_RTS
-Text Label 6950 6200 2    50   ~ 0
-FMU_USART2_TX
-Text Label 6950 6300 2    50   ~ 0
-FMU_USART2_RX
+Text Label 1700 1650 0    50   ~ 0
+STM_CTS_TELEM_RTS_USART2
 Text Label 1700 1550 0    50   ~ 0
-FMU_USART2_CTS
-Text Label 1700 1650 0    50   ~ 0
-FMU_USART2_RTS
+STM_RTS_TELEM_CTS_USART2
+Text Label 1700 1850 0    50   ~ 0
+STM_TX_TELEM_RX_USART2
 Text Label 1700 1750 0    50   ~ 0
-FMU_USART2_TX
-Text Label 1700 1850 0    50   ~ 0
-FMU_USART2_RX
+STM_RX_TELEM_TX_USART2
 Text Label 8750 2800 0    50   ~ 0
 SENSOR_SCK
@@
 Text Label 14150 3250 2    50   ~ 0
 STM_RX_GPS_TX_USART6
+Text Label 6950 6000 2    50   ~ 0
+STM_CTS_TELEM_RTS_USART2
+Text Label 6950 6100 2    50   ~ 0
+STM_RTS_TELEM_CTS_USART2
+Text Label 6950 6200 2    50   ~ 0
+STM_TX_TELEM_RX_USART2
+Text Label 6950 6300 2    50   ~ 0
+STM_RX_TELEM_TX_USART2
+NoConn ~ 8750 4100
+NoConn ~ 8750 4200
+NoConn ~ 8750 3300
+NoConn ~ 6950 4100
+NoConn ~ 6950 4000
+NoConn ~ 8750 4600
+NoConn ~ 8750 4700
+NoConn ~ 8750 6200
 $EndSCHEMATC
